File: Power Distribution Board.kicad_pcb (KiCad board)
At the start: 2 copper layers, 13 parts, among them J1 XT90PW-F, J2 XT90PW-F, J3 XT90PW-F, J4 XT90PW-F, J6 XT90PW-F, U1 LM2576HVS-5

Commit message: Version as of 10-16
Parts:
- added L1: 10uH, Inductor_SMD:L_APV_APH1030, F.Cu at (234.5, 83.7)
- U1: value LM2576HVS-5 -> LM76003RNPR; footprint Package_TO_SOT_SMD:TO-263-5_TabPin3 -> LM76003RNPT:RNP0030B
- moved U1 52.6 mm to (165.1, 90.5)
Connections:
- C1 pad 2: Net-(J1-+) -> GND
- C2 pad 2: Net-(J1-+) -> GND
- C3 pad 2: Net-(J1-+) -> GND
- C4 pad 2: Net-(J1-+) -> GND
- C5 pad 2: Net-(J1-+) -> GND
- CR1 pad 2: Net-(J1-+) -> GND
- J1 pad 1: Net-(J1-+) -> GND
- J2 pad 3: Net-(J1-+) -> GND
- J3 pad 3: Net-(J1-+) -> GND
- J4 pad 3: Net-(J1-+) -> GND
- U1 pad 1: Net-(J1--) -> Net-(Cboot1-Pad2)
- U1 pad 2: unconnected-(U1-OUT-Pad2) -> Net-(Cboot1-Pad2)
- U1 pad 3: GND -> Net-(Cboot1-Pad2)
- U1 pad 4: unconnected-(U1-FB-Pad4) -> Net-(Cboot1-Pad2)
- U1 pad 5: unconnected-(U1-~{ON}/OFF-Pad5) -> Net-(Cboot1-Pad2)
